File: green_storm.kicad_sch (KiCad schematic)
At the start: 28 parts, among them J1 USB_B_Micro, J2 Conn_01x04, J3 Conn_01x04, J4 Conn_01x04, SW1 SW_SPDT, U1 STM32F103C8T6, U2 AMS1117-3.3, Y1 16Mhz

Commit message: Updatd Schematic in KiCad
Parts:
- renumbered C12 to C1, C8 to C10, C9 to C11, C10 to C12, C11 to C13, C13 to C2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
Other:
- moved on the sheet: J2
