File: green_storm.kicad_sch (KiCad schematic)
At the start: 28 parts, among them J1 USB_B_Micro, J2 Conn_01x04, J3 Conn_01x04, J4 Conn_01x04, SW1 SW_SPDT, U1 AMS1117-3.3, U2 STM32F103C8T6, Y1 16Mhz

Commit message: Revised eschema
Connections:
- net at R3.2, U2.33 (PA12): now also J1.3 (D+); no longer J1.2 (D-)
- net at U2.32 (PA11): now also J1.2 (D-); no longer J1.3 (D+)
Other:
- moved on the sheet: J1
Changed lines of the file:
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@@
   (junction (at 83.82 96.52) (diameter 0) (color 0 0 0 0)
   )
+  (junction (at 107.95 96.52) (diameter 0) (color 0 0 0 0)
+  )
+  (junction (at 139.7 27.94) (diameter 0) (color 0 0 0 0)
+  )
+  (junction (at 139.7 41.91) (diameter 0) (color 0 0 0 0)
+  )
+  (junction (at 127 27.94) (diameter 0) (color 0 0 0 0)
+  )
+  (junction (at 83.82 114.3) (diameter 0) (color 0 0 0 0)
+  )
+  (junction (at 207.01 27.94) (diameter 0) (color 0 0 0 0)
+  )
+  (junction (at 195.58 27.94) (diameter 0) (color 0 0 0 0)
+  )
+  (junction (at 107.95 106.68) (diameter 0) (color 0 0 0 0)
+  )
+  (junction (at 128.27 124.46) (diameter 0) (color 0 0 0 0)
+  )
+  (junction (at 36.83 71.12) (diameter 0) (color 0 0 0 0)
+  )
+  (junction (at 83.82 106.68) (diameter 0) (color 0 0 0 0)
+  )
+  (junction (at 153.67 27.94) (diameter 0) (color 0 0 0 0)
+  )
   (junction (at 224.79 82.55) (diameter 0) (color 0 0 0 0)
-  )
-  (junction (at 107.95 96.52) (diameter 0) (color 0 0 0 0)
-  )
-  (junction (at 139.7 27.94) (diameter 0) (color 0 0 0 0)
-  )
-  (junction (at 139.7 41.91) (diameter 0) (color 0 0 0 0)
-  )
-  (junction (at 127 27.94) (diameter 0) (color 0 0 0 0)
-  )
-  (junction (at 83.82 114.3) (diameter 0) (color 0 0 0 0)
-  )
-  (junction (at 207.01 27.94) (diameter 0) (color 0 0 0 0)
-  )
-  (junction (at 195.58 27.94) (diameter 0) (color 0 0 0 0)
-  )
-  (junction (at 107.95 106.68) (diameter 0) (color 0 0 0 0)
-  )
-  (junction (at 128.27 124.46) (diameter 0) (color 0 0 0 0)
-  )
-  (junction (at 36.83 71.12) (diameter 0) (color 0 0 0 0)
-  )
-  (junction (at 83.82 106.68) (diameter 0) (color 0 0 0 0)
-  )
-  (junction (at 153.67 27.94) (diameter 0) (color 0 0 0 0)
   )
   (junction (at 187.96 40.64) (diameter 0) (color 0 0 0 0)
@@
   (no_connect (at 172.72 87.63))
   (no_connect (at 172.72 82.55))
-  (no_connect (at 231.14 80.01))
+  (no_connect (at 233.68 77.47))
   (no_connect (at 172.72 100.33))
   (no_connect (at 172.72 74.93))
@@
   (no_connect (at 205.74 67.31))
   (no_connect (at 172.72 72.39))
-  (no_connect (at 241.3 74.93))
+  (no_connect (at 243.84 72.39))
   (no_connect (at 205.74 69.85))
   (no_connect (at 205.74 52.07))
@@
     (stroke (width 0) (type default))
   )
+  (wire (pts (xy 205.74 80.01) (xy 233.68 80.01))
+    (stroke (width 0) (type default))
+  )
   (wire (pts (xy 66.04 50.8) (xy 66.04 55.88))
     (stroke (width 0) (type default))
@@
     (stroke (width 0) (type default))
   )
-  (wire (pts (xy 224.79 82.55) (xy 231.14 82.55))
-    (stroke (width 0) (type default))
-  )
   (wire (pts (xy 118.11 78.74) (xy 118.11 83.82))
     (stroke (width 0) (type default))
@@
     (stroke (width 0) (type default))
   )
-  (wire (pts (xy 238.76 71.12) (xy 238.76 74.93))
+  (wire (pts (xy 241.3 68.58) (xy 241.3 72.39))
     (stroke (width 0) (type default))
   )
@@
     (stroke (width 0) (type default))
   )
-  (wire (pts (xy 205.74 80.01) (xy 219.71 80.01))
-    (stroke (width 0) (type default))
-  )
   (wire (pts (xy 128.27 151.13) (xy 128.27 157.48))
     (stroke (width 0) (type default))
@@
     (stroke (width 0) (type default))
   )
-  (wire (pts (xy 224.79 90.17) (xy 224.79 93.98))
+  (wire (pts (xy 229.87 87.63) (xy 229.87 91.44))
     (stroke (width 0) (type default))
   )
@@
     (stroke (width 0) (type default))
   )
-  (wire (pts (xy 231.14 85.09) (xy 219.71 85.09))
-    (stroke (width 0) (type default))
-  )
   (wire (pts (xy 83.82 106.68) (xy 107.95 106.68))
     (stroke (width 0) (type default))
@@
     (stroke (width 0) (type default))
   )
+  (wire (pts (xy 224.79 82.55) (xy 233.68 82.55))
+    (stroke (width 0) (type default))
+  )
   (wire (pts (xy 83.82 96.52) (xy 83.82 106.68))
     (stroke (width 0) (type default))
@@
     (stroke (width 0) (type default))
   )
-  (wire (pts (xy 219.71 85.09) (xy 219.71 80.01))
-    (stroke (width 0) (type default))
-  )
   (wire (pts (xy 49.53 71.12) (xy 66.04 71.12))
     (stroke (width 0) (type default))
@@
     (stroke (width 0) (type default))
   )
-  (wire (pts (xy 224.79 90.17) (xy 231.14 90.17))
+  (wire (pts (xy 229.87 87.63) (xy 233.68 87.63))
     (stroke (width 0) (type default))
   )
@@
     (effects (font (size 2.5 2.5) (thickness 0.4) bold) (justify left bottom))
   )
-  (text "USB App note AN879" (at 234.95 64.77 0)
+  (text "USB App note AN879" (at 233.68 63.5 0)
     (effects (font (size 1.27 1.27) bold) (justify left bottom))
   )
@@
     )
   )
-  (symbol (lib_id "power:VBUS") (at 224.79 93.98 0) (mirror x) (unit 1)
+  (symbol (lib_id "power:VBUS") (at 229.87 91.44 0) (mirror x) (unit 1)
     (in_bom yes) (on_board yes) (dnp no)
-    (property "Reference" "#PWR014" (at 224.79 90.17 0)
-      (effects (font (size 1.27 1.27)) hide)
-    )
-    (property "Value" "VBUS" (at 224.79 97.79 0)
-      (effects (font (size 1.27 1.27)))
-    )
-    (property "Footprint" "" (at 224.79 93.98 0)
-      (effects (font (size 1.27 1.27)) hide)
-    )
-    (property "Datasheet" "" (at 224.79 93.98 0)
+    (property "Reference" "#PWR014" (at 229.87 87.63 0)
+      (effects (font (size 1.27 1.27)) hide)
+    )
+    (property "Value" "VBUS" (at 229.87 95.25 0)
+      (effects (font (size 1.27 1.27)))
+    )
+    (property "Footprint" "" (at 229.87 91.44 0)
+      (effects (font (size 1.27 1.27)) hide)
+    )
+    (property "Datasheet" "" (at 229.87 91.44 0)
       (effects (font (size 1.27 1.27)) hide)
     )
@@
     )
   )
-  (symbol (lib_name "GND_1") (lib_id "power:GND") (at 238.76 71.12 180) (unit 1)
+  (symbol (lib_name "GND_1") (lib_id "power:GND") (at 241.3 68.58 180) (unit 1)
     (in_bom yes) (on_board yes) (dnp no)
-    (property "Reference" "#PWR012" (at 238.76 64.77 0)
-      (effects (font (size 1.27 1.27)) hide)
-    )
-    (property "Value" "GND" (at 238.76 66.04 0)
-      (effects (font (size 1.27 1.27)) hide)
-    )
-    (property "Footprint" "" (at 238.76 71.12 0)
-      (effects (font (size 1.27 1.27)) hide)
-    )
-    (property "Datasheet" "" (at 238.76 71.12 0)
+    (property "Reference" "#PWR012" (at 241.3 62.23 0)
+      (effects (font (size 1.27 1.27)) hide)
+    )
+    (property "Value" "GND" (at 241.3 63.5 0)
+      (effects (font (size 1.27 1.27)) hide)
+    )
+    (property "Footprint" "" (at 241.3 68.58 0)
+      (effects (font (size 1.27 1.27)) hide)
+    )
+    (property "Datasheet" "" (at 241.3 68.58 0)
       (effects (font (size 1.27 1.27)) hide)
     )
@@
     )
   )
-  (symbol (lib_id "Connector:USB_B_Micro") (at 238.76 85.09 180) (unit 1)
+  (symbol (lib_id "Connector:USB_B_Micro") (at 241.3 82.55 180) (unit 1)
     (in_bom yes) (on_board yes) (dnp no)
-    (property "Reference" "J1" (at 238.76 97.79 0)
-      (effects (font (size 1.27 1.27)))
-    )
-    (property "Value" "USB_B_Micro" (at 238.76 95.25 0)
-      (effects (font (size 1.27 1.27)))
-    )
-    (property "Footprint" "" (at 234.95 83.82 0)
-      (effects (font (size 1.27 1.27)) hide)
-    )
-    (property "Datasheet" "~" (at 234.95 83.82 0)
-      (effects (font (size 1.27 1.27)) hide)
-    )
+    (property "Reference" "J1" (at 241.3 95.25 0)
+      (effects (font (size 1.27 1.27)))
+    )
+    (property "Value" "USB_B_Micro" (at 241.3 92.71 0)
+      (effects (font (size 1.27 1.27)))
+    )
+    (property "Footprint" "" (at 237.49 81.28 0)
+      (effects (font (size 1.27 1.27)) hide)
+    )
+    (property "Datasheet" "~" (at 237.49 81.28 0)
+      (effects (font (size 1.27 1.27)) hide)
+    )
