File: green_storm.kicad_sch (KiCad schematic)
At the start: 28 parts, among them J1 USB_B_Micro, J2 Conn_01x04, J3 Conn_01x04, J4 Conn_01x04, SW1 SW_SPDT, U1 AMS1117-3.3, U2 STM32F103C8T6, Y1 16Mhz

Commit message: Revised schematic - removed sneaky wire
Connections:
- net GND: no longer C12.1, C13.1, U2.5 (PD0), U2.6 (PD1), Y1.1, Y1.3
- new net: C12.1, U2.5 (PD0), Y1.1
- new net: C13.1, U2.6 (PD1), Y1.3
Changed lines of the file:
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@@
   (junction (at 195.58 27.94) (diameter 0) (color 0 0 0 0)
   )
-  (junction (at 107.95 106.68) (diameter 0) (color 0 0 0 0)
-  )
   (junction (at 128.27 124.46) (diameter 0) (color 0 0 0 0)
   )
   (junction (at 36.83 71.12) (diameter 0) (color 0 0 0 0)
-  )
-  (junction (at 83.82 106.68) (diameter 0) (color 0 0 0 0)
   )
   (junction (at 153.67 27.94) (diameter 0) (color 0 0 0 0)
@@
     (stroke (width 0) (type default))
   )
-  (wire (pts (xy 83.82 114.3) (xy 83.82 106.68))
-    (stroke (width 0) (type default))
-  )
   (wire (pts (xy 167.64 39.37) (xy 167.64 41.91))
     (stroke (width 0) (type default))
@@
   )
   (wire (pts (xy 138.43 132.08) (xy 138.43 133.35))
-    (stroke (width 0) (type default))
-  )
-  (wire (pts (xy 83.82 106.68) (xy 107.95 106.68))
     (stroke (width 0) (type default))
   )
@@
       (effects (font (size 1.27 1.27)) hide)
     )
-    (property "Value" "VBUS" (at 257.81 93.98 0)
+    (property "Value" "VBUS" (at 243.84 95.25 0)
       (effects (font (size 1.27 1.27)))
     )

Commit message: Half point of PCB layout
Parts:
- C1, C2: footprint (none) -> Capacitor_SMD:C_0805_2012Metric
- C10, C11, C12, C13, C4, C5, C6, C7, C8, C9: footprint (none) -> Capacitor_SMD:C_0402_1005Metric
- C3: footprint (none) -> Capacitor_SMD:C_0603_1608Metric
- D1: footprint (none) -> LED_SMD:LED_0603_1608Metric
- FB1: footprint (none) -> Inductor_SMD:L_0603_1608Metric
- J1: footprint (none) -> Connector_USB:USB_Micro-B_Wuerth_629105150521
- J2, J3: footprint (none) -> Connector_PinHeader_2.54mm:PinHeader_1x04_P2.54mm_Vertical
- J4: footprint (none) -> Connector_PinHeader_2.00mm:PinHeader_1x04_P2.00mm_Vertical
- R1, R2, R3, R4, R5: footprint (none) -> Resistor_SMD:R_0402_1005Metric
- SW1: footprint (none) -> Button_Switch_SMD:SW_SPDT_PCM12
- Y1: footprint (none) -> Crystal:Crystal_SMD_3225-4Pin_3.2x2.5mm
Changed lines of the file:
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@@
       (effects (font (size 1.27 1.27)) (justify left))
     )
-    (property "Footprint" "" (at 136.652 139.7 90)
+    (property "Footprint" "Resistor_SMD:R_0402_1005Metric" (at 136.652 139.7 90)
       (effects (font (size 1.27 1.27)) hide)
     )
@@
       (effects (font (size 1.27 1.27)) (justify left))
     )
-    (property "Footprint" "" (at 154.6352 39.37 0)
+    (property "Footprint" "Capacitor_SMD:C_0402_1005Metric" (at 154.6352 39.37 0)
       (effects (font (size 1.27 1.27)) hide)
     )
@@
       (effects (font (size 1.27 1.27)) (justify left))
     )
-    (property "Footprint" "" (at 223.52 106.68 0)
+    (property "Footprint" "Connector_PinHeader_2.54mm:PinHeader_1x04_P2.54mm_Vertical" (at 223.52 106.68 0)
       (effects (font (size 1.27 1.27)) hide)
     )
@@
       (effects (font (size 1.27 1.27)) (justify left))
     )
-    (property "Footprint" "" (at 64.262 59.69 90)
+    (property "Footprint" "Resistor_SMD:R_0402_1005Metric" (at 64.262 59.69 90)
       (effects (font (size 1.27 1.27)) hide)
     )
@@
       (effects (font (size 1.27 1.27)) (justify left))
     )
-    (property "Footprint" "" (at 216.8652 35.56 0)
+    (property "Footprint" "Capacitor_SMD:C_0402_1005Metric" (at 216.8652 35.56 0)
       (effects (font (size 1.27 1.27)) hide)
     )
@@
       (effects (font (size 1.27 1.27)) (justify left))
     )
-    (property "Footprint" "" (at 229.5652 35.56 0)
+    (property "Footprint" "Capacitor_SMD:C_0402_1005Metric" (at 229.5652 35.56 0)
       (effects (font (size 1.27 1.27)) hide)
     )
@@
       (effects (font (size 1.27 1.27)) (justify left))
     )
-    (property "Footprint" "" (at 168.6052 39.37 0)
+    (property "Footprint" "Capacitor_SMD:C_0402_1005Metric" (at 168.6052 39.37 0)
       (effects (font (size 1.27 1.27)) hide)
     )
@@
       (effects (font (size 1.27 1.27)) (justify left))
     )
-    (property "Footprint" "" (at 140.6652 39.37 0)
+    (property "Footprint" "Capacitor_SMD:C_0402_1005Metric" (at 140.6652 39.37 0)
       (effects (font (size 1.27 1.27)) hide)
     )
@@
       (effects (font (size 1.27 1.27)) (justify left))
     )
-    (property "Footprint" "" (at 122.8852 59.69 0)
+    (property "Footprint" "Capacitor_SMD:C_0402_1005Metric" (at 122.8852 59.69 0)
       (effects (font (size 1.27 1.27)) hide)
     )
@@
       (effects (font (size 1.27 1.27)))
     )
-    (property "Footprint" "" (at 93.98 96.52 0)
+    (property "Footprint" "Crystal:Crystal_SMD_3225-4Pin_3.2x2.5mm" (at 93.98 96.52 0)
       (effects (font (size 1.27 1.27)) hide)
     )
@@
       (effects (font (size 1.27 1.27)))
     )
-    (property "Footprint" "" (at 54.61 50.8 0)
+    (property "Footprint" "LED_SMD:LED_0603_1608Metric" (at 54.61 50.8 0)
       (effects (font (size 1.27 1.27)) hide)
     )
@@
       (effects (font (size 1.27 1.27)) (justify left))
     )
-    (property "Footprint" "" (at 23.8252 71.12 0)
+    (property "Footprint" "Capacitor_SMD:C_0805_2012Metric" (at 23.8252 71.12 0)
       (effects (font (size 1.27 1.27)) hide)
     )
@@
       (effects (font (size 1.27 1.27)) (justify left))
     )
-    (property "Footprint" "" (at 223.012 74.93 90)
+    (property "Footprint" "Resistor_SMD:R_0402_1005Metric" (at 223.012 74.93 90)
       (effects (font (size 1.27 1.27)) hide)
     )
@@
       (effects (font (size 1.27 1.27)))
     )
-    (property "Footprint" "" (at 146.05 77.978 90)
+    (property "Footprint" "Resistor_SMD:R_0402_1005Metric" (at 146.05 77.978 90)
       (effects (font (size 1.27 1.27)) hide)
     )
@@
       (effects (font (size 1.27 1.27)))
     )
-    (property "Footprint" "" (at 251.46 81.28 0)
+    (property "Footprint" "Connector_USB:USB_Micro-B_Wuerth_629105150521" (at 251.46 81.28 0)
       (effects (font (size 1.27 1.27)) hide)
     )
@@
       (effects (font (size 1.27 1.27)))
     )
-    (property "Footprint" "" (at 123.19 76.2 0)
+    (property "Footprint" "Button_Switch_SMD:SW_SPDT_PCM12" (at 123.19 76.2 0)
       (effects (font (size 1.27 1.27)) hide)
     )
@@
       (effects (font (size 1.27 1.27)) (justify left))
     )
-    (property "Footprint" "" (at 108.9152 114.3 0)
+    (property "Footprint" "Capacitor_SMD:C_0402_1005Metric" (at 108.9152 114.3 0)
       (effects (font (size 1.27 1.27)) hide)
     )
@@
       (effects (font (size 1.27 1.27)) (justify left))
     )
-    (property "Footprint" "" (at 84.7852 114.3 0)
+    (property "Footprint" "Capacitor_SMD:C_0402_1005Metric" (at 84.7852 114.3 0)
       (effects (font (size 1.27 1.27)) hide)
     )
@@
       (effects (font (size 1 1)) (justify left))
     )
-    (property "Footprint" "" (at 123.19 119.38 0)
+    (property "Footprint" "Connector_PinHeader_2.54mm:PinHeader_1x04_P2.54mm_Vertical" (at 123.19 119.38 0)
       (effects (font (size 1.27 1.27)) hide)
     )
@@
       (effects (font (size 1.27 1.27)) (justify left))
     )
-    (property "Footprint" "" (at 50.4952 71.12 0)
+    (property "Footprint" "Capacitor_SMD:C_0805_2012Metric" (at 50.4952 71.12 0)
       (effects (font (size 1.27 1.27)) hide)
     )
@@
       (effects (font (size 1.27 1.27)) (justify left))
     )
-    (property "Footprint" "" (at 127.9652 39.37 0)
+    (property "Footprint" "Capacitor_SMD:C_0402_1005Metric" (at 127.9652 39.37 0)
       (effects (font (size 1.27 1.27)) hide)
     )
@@
       (effects (font (size 1.27 1.27)) (justify left))
     )
-    (property "Footprint" "" (at 113.9952 39.37 0)
+    (property "Footprint" "Capacitor_SMD:C_0603_1608Metric" (at 113.9952 39.37 0)
       (effects (font (size 1.27 1.27)) hide)
     )
@@
       (effects (font (size 1.27 1.27)) (justify left))
     )
-    (property "Footprint" "" (at 254.9652 35.56 0)
+    (property "Footprint" "Capacitor_SMD:C_0402_1005Metric" (at 254.9652 35.56 0)
       (effects (font (size 1.27 1.27)) hide)
     )
@@
       (effects (font (size 1.27 1.27)) (justify left))
     )
-    (property "Footprint" "" (at 146.812 139.7 90)
+    (property "Footprint" "Resistor_SMD:R_0402_1005Metric" (at 146.812 139.7 90)
       (effects (font (size 1.27 1.27)) hide)
     )
@@
       (effects (font (size 1 1)) (justify left))
     )
-    (property "Footprint" "" (at 123.19 146.05 0)
+    (property "Footprint" "Connector_PinHeader_2.00mm:PinHeader_1x04_P2.00mm_Vertical" (at 123.19 146.05 0)
       (effects (font (size 1.27 1.27)) hide)
     )
@@
       (effects (font (size 1.27 1.27)))
     )
-    (property "Footprint" "" (at 242.57 29.718 90)
-      (effects (font (size 1.27 1.27)) hide)
-    )
+    (property "Footprint" "Inductor_SMD:L_0603_1608Metric" (at 242.57 29.718 90)
+      (effects (font (size 1.27 1.27)) hide)
+    )

Commit message: Routing half-way complete
Parts:
- added H1, H2, H3, H4: MountingHole, MountingHole:MountingHole_2.2mm_M2, symbol Mechanical:MountingHole
Other:
- note added: "M2"
- note added: "Mounting Holes"
Changed lines of the file:
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@@
+    (stroke (width 0) (type default))
+  )
+  (polyline (pts (xy 46.99 134.62) (xy 15.24 134.62))
     (stroke (width 0) (type default))
   )
@@
     (stroke (width 0) (type default))
   )
+  (polyline (pts (xy 46.99 166.37) (xy 15.24 166.37))
+    (stroke (width 0) (type default))
+  )
   (wire (pts (xy 228.6 38.1) (xy 228.6 41.91))
     (stroke (width 0) (type default))
@@
     (stroke (width 0) (type default))
   )
+  (polyline (pts (xy 15.24 166.37) (xy 15.24 134.62))
+    (stroke (width 0) (type default))
+  )
   (wire (pts (xy 205.74 82.55) (xy 224.79 82.55))
     (stroke (width 0) (type default))
@@
     (stroke (width 0) (type default))
   )
+  (polyline (pts (xy 46.99 134.62) (xy 46.99 135.89))
+    (stroke (width 0) (type default))
+  )
   (wire (pts (xy 195.58 27.94) (xy 195.58 46.99))
     (stroke (width 0) (type default))
@@
   )
   (wire (pts (xy 163.83 107.95) (xy 163.83 148.59))
+    (stroke (width 0) (type default))
+  )
+  (polyline (pts (xy 46.99 166.37) (xy 46.99 134.62))
     (stroke (width 0) (type default))
   )
@@
     (effects (font (size 1.27 1.27) bold) (justify left bottom))
   )
+  (text "Mounting Holes" (at 16.51 133.35 0)
+    (effects (font (size 2 2) (thickness 0.4) bold) (justify left bottom))
+  )
   (text "SWDI0" (at 207.01 85.09 0)
     (effects (font (size 1 1)) (justify left bottom))
@@
     (effects (font (size 1 1) bold) (justify left bottom))
   )
+  (text "M2" (at 16.51 170.18 0)
+    (effects (font (size 1.27 1.27) bold) (justify left bottom))
+  )
   (text "1 x 100nF per VDD Pin" (at 134.62 25.4 0)
     (effects (font (size 0.75 0.75) bold) (justify left bottom))
@@
   (text "SW_BOOT0" (at 130.81 76.2 0)
     (effects (font (size 1.27 1.27)) (justify left bottom))
+  )
+  (symbol (lib_id "Mechanical:MountingHole") (at 19.05 153.67 0) (unit 1)
+    (in_bom yes) (on_board yes) (dnp no) (fields_autoplaced)
+    (property "Reference" "H3" (at 21.59 152.4 0)
+      (effects (font (size 1.27 1.27)) (justify left))
+    )
+    (property "Value" "MountingHole" (at 21.59 154.94 0)
+      (effects (font (size 1.27 1.27)) (justify left))
+    )
+    (property "Footprint" "MountingHole:MountingHole_2.2mm_M2" (at 19.05 153.67 0)
+      (effects (font (size 1.27 1.27)) hide)
+    )
+    (property "Datasheet" "~" (at 19.05 153.67 0)
+      (effects (font (size 1.27 1.27)) hide)
+    )
+    (instances
+      (project "green_storm"
+        (path "/3cfe805b-14ec-42f0-9564-1ea3fdf6f438"
+          (reference "H3") (unit 1)
+        )
+      )
+    )
   )
   (symbol (lib_name "R_2") (lib_id "Device:R") (at 138.43 139.7 0) (unit 1)
@@
     )
   )
+  (symbol (lib_id "Mechanical:MountingHole") (at 19.05 160.02 0) (unit 1)
+    (in_bom yes) (on_board yes) (dnp no) (fields_autoplaced)
+    (property "Reference" "H4" (at 21.59 158.75 0)
+      (effects (font (size 1.27 1.27)) (justify left))
+    )
+    (property "Value" "MountingHole" (at 21.59 161.29 0)
+      (effects (font (size 1.27 1.27)) (justify left))
+    )
+    (property "Footprint" "MountingHole:MountingHole_2.2mm_M2" (at 19.05 160.02 0)
+      (effects (font (size 1.27 1.27)) hide)
+    )
+    (property "Datasheet" "~" (at 19.05 160.02 0)
+      (effects (font (size 1.27 1.27)) hide)
+    )
+    (instances
+      (project "green_storm"
+        (path "/3cfe805b-14ec-42f0-9564-1ea3fdf6f438"
+          (reference "H4") (unit 1)
+        )
+      )
+    )
+  )
   (symbol (lib_id "power:PWR_FLAG") (at 207.01 27.94 0) (unit 1)
     (in_bom yes) (on_board yes) (dnp no) (fields_autoplaced)
@@
     )
   )
+  (symbol (lib_id "Mechanical:MountingHole") (at 19.05 140.97 0) (unit 1)
+    (in_bom yes) (on_board yes) (dnp no)
+    (property "Reference" "H1" (at 21.59 139.7 0)
+      (effects (font (size 1.27 1.27)) (justify left))
+    )
+    (property "Value" "MountingHole" (at 21.59 142.24 0)
+      (effects (font (size 1.27 1.27)) (justify left))
+    )
+    (property "Footprint" "MountingHole:MountingHole_2.2mm_M2" (at 19.05 140.97 0)
+      (effects (font (size 1.27 1.27)) hide)
+    )
+    (property "Datasheet" "~" (at 19.05 140.97 0)
+      (effects (font (size 1.27 1.27)) hide)
+    )
+    (instances
+      (project "green_storm"
+        (path "/3cfe805b-14ec-42f0-9564-1ea3fdf6f438"
+          (reference "H1") (unit 1)
+        )
+      )
+    )
+  )
   (symbol (lib_id "Device:C") (at 121.92 55.88 0) (unit 1)
     (in_bom yes) (on_board yes) (dnp no) (fields_autoplaced)
@@
         )
       )
+    )
+  )
+  (symbol (lib_id "Mechanical:MountingHole") (at 19.05 147.32 0) (unit 1)
+    (in_bom yes) (on_board yes) (dnp no) (fields_autoplaced)
+    (property "Reference" "H2" (at 21.59 146.05 0)
+      (effects (font (size 1.27 1.27)) (justify left))
+    )
+    (property "Value" "MountingHole" (at 21.59 148.59 0)
+      (effects (font (size 1.27 1.27)) (justify left))
+    )
+    (property "Footprint" "MountingHole:MountingHole_2.2mm_M2" (at 19.05 147.32 0)
+      (effects (font (size 1.27 1.27)) hide)
+    )
+    (property "Datasheet" "~" (at 19.05 147.32 0)
+      (effects (font (size 1.27 1.27)) hide)
+    )
+    (instances
+      (project "green_storm"
+        (path "/3cfe805b-14ec-42f0-9564-1ea3fdf6f438"
+          (reference "H2") (unit 1)
+        )
+      )

Commit message: Off to Manufacturing
Parts:
- J4: footprint Connector_PinHeader_2.00mm:PinHeader_1x04_P2.00mm_Vertical -> Connector_PinHeader_2.54mm:PinHeader_1x04_P2.54mm_Vertical
Connections:
- net GND: now also J1.6 (Shield)
- no-connect marks 29 -> 28
Changed lines of the file:
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@@
   (no_connect (at 205.74 67.31))
   (no_connect (at 172.72 72.39))
-  (no_connect (at 257.81 72.39))
   (no_connect (at 205.74 69.85))
   (no_connect (at 205.74 52.07))
@@
     (stroke (width 0) (type default))
   )
+  (wire (pts (xy 257.81 68.58) (xy 257.81 72.39))
+    (stroke (width 0) (type default))
+  )
   (wire (pts (xy 83.82 114.3) (xy 93.98 114.3))
     (stroke (width 0) (type default))
@@
         (path "/3cfe805b-14ec-42f0-9564-1ea3fdf6f438"
           (reference "C11") (unit 1)
+        )
+      )
+    )
+  )
+  (symbol (lib_name "GND_1") (lib_id "power:GND") (at 257.81 68.58 180) (unit 1)
+    (in_bom yes) (on_board yes) (dnp no)
+    (property "Reference" "#PWR013" (at 257.81 62.23 0)
+      (effects (font (size 1.27 1.27)) hide)
+    )
+    (property "Value" "GND" (at 257.81 63.5 0)
+      (effects (font (size 1.27 1.27)) hide)
+    )
+    (property "Footprint" "" (at 257.81 68.58 0)
+      (effects (font (size 1.27 1.27)) hide)
+    )
+    (property "Datasheet" "" (at 257.81 68.58 0)
+      (effects (font (size 1.27 1.27)) hide)
+    )
+    (pin "1")
+    (instances
+      (project "green_storm"
+        (path "/3cfe805b-14ec-42f0-9564-1ea3fdf6f438"
+          (reference "#PWR013") (unit 1)
         )
       )
@@
       (effects (font (size 1 1)) (justify left))
     )
-    (property "Footprint" "Connector_PinHeader_2.00mm:PinHeader_1x04_P2.00mm_Vertical" (at 123.19 146.05 0)
-      (effects (font (size 1.27 1.27)) hide)
-    )
+    (property "Footprint" "Connector_PinHeader_2.54mm:PinHeader_1x04_P2.54mm_Vertical" (at 123.19 146.05 0)
+      (effects (font (size 1.27 1.27)) hide)
+    )
